Commit message: Change Project Name

File: description/gazebo_control.xacro (robot description, xacro)
@@ -8,7 +8,7 @@
             <wheel_separation>0.297</wheel_separation>
             <wheel_diameter>0.066</wheel_diameter>
-            <!-- Limits -->
-            <max_wheel_torque>200</max_wheel_torque>
-            <max_wheel_acceleration>10.0</max_wheel_acceleration>
+            <!-- Limits  가제보 속도 조절 코드(추후에 실제로봇이랑 가제보랑 비슷하게 해야함) -->
+            <max_wheel_torque>800</max_wheel_torque>
+            <max_wheel_acceleration>80.0</max_wheel_acceleration>
             <!-- Output -->
             <odometry_frame>odom</odometry_frame>

File: description/ros2_control.xacro (robot description, xacro)
@@ -1,5 +1,33 @@
 <?xml version="1.0"?>
 <robot xmlns:xacro="http://www.ros.org/wiki/xacro">
-    <ros2_control name = "GazeboSystem" type = "system">
+    <ros2_control name = "RealRobot" type = "system">
+        <hardware>
+            <plugin>diffdrive_arduino/DiffDriveArduino</plugin>
+            <param name="left_wheel_name">left_wheel_joint</param>
+            <param name="right_wheel_name">right_wheel_joint</param>
+            <param name="loop_rate">30</param>
+            <param name="device">/dev/ttyUSB0</param>
+            <param name="baud_rate">57600</param>
+            <param name="timeout">1000</param>
+            <param name="enc_counts_per_rev">30000</param>  <!-- 실제바퀴와 시뮬레이션 상 바퀴 조절할대 값 수정(작을수록 빨리돌고, 클수록 느리게 돎)-->
+        </hardware>
+        <joint name = "left_wheel_joint">
+            <command_interface name = "velocity">
+                <param name = "min">-10</param>
+                <param name = "max">10</param>
+            </command_interface>
+            <state_interface name = "velocity"/>
+            <state_interface name = "position"/>
+        </joint>
+        <joint name = "right_wheel_joint">
+            <command_interface name = "velocity">
+                <param name = "min">-10</param>
+                <param name = "max">10</param>
+            </command_interface>
+            <state_interface name = "velocity"/>
+            <state_interface name = "position"/>
+        </joint>
+    </ros2_control>
+    <!-- <ros2_control name = "GazeboSystem" type = "system">
         <hardware>
             <plugin>gazebo_ros2_control/GazeboSystem</plugin>
@@ -21,5 +49,5 @@
             <state_interface name = "position"/>
         </joint>
-    </ros2_control>
+    </ros2_control> -->
     <gazebo>
         <plugin name="gazebo_ros2_control" filename="libgazebo_ros2_control.so">
